File: PCB v22.brd (EAGLE design)
At the start: 100 x 100 mm, 166 parts

Commit message: usb routing
Connections:
- net N$7 renamed USB_N
- net N$8 renamed USB_P
Routing:
- net USB_N: track 48.5 -> 51.4 mm
- net USB_P: track 50.2 -> 47.5 mm
- net GND: track 328.7 -> 329.6 mm
- net 5V0: track 155.8 -> 156.6 mm
